File: Trial.brd (EAGLE design)
At the start: 130.8 x 143.2 mm, 11 parts

Commit message: Edited schematic file
Other:
- board size 130.8 x 143.2 mm -> 130.8 x 122.9 mm
Changed lines of the file:
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@@
 </layers>
 <board>
-<fusionsync huburn="a.YnVzaW5lc3M6bXlpdHU3Mzc" projecturn="a.YnVzaW5lc3M6bXlpdHU3MzcjMjAyMDEyMjYzNjU2MjcyNTY" f3durn="urn:adsk.wipprod:dm.lineage:BmzR0BmFQhKo_aDMTO62Ig" pcbguid="" lastpulledtime="" lastsyncedchangeguid="" latestrevisionid="458f3546-b32b-41f4-945d-214eebd3752f" lastsyncedrevisionid="458f3546-b32b-41f4-945d-214eebd3752f" lastboardhashguid="dd785595-ab13-82c8-a0c8-971baf9ee58e" lastpushedtime="2021-03-23T11:39:58Z" linktopcb3d="true"/>
+<fusionsync huburn="a.YnVzaW5lc3M6bXlpdHU3Mzc" projecturn="a.YnVzaW5lc3M6bXlpdHU3MzcjMjAyMDEyMjYzNjU2MjcyNTY" f3durn="urn:adsk.wipprod:dm.lineage:BmzR0BmFQhKo_aDMTO62Ig" pcbguid="" lastpulledtime="" lastsyncedchangeguid="" latestrevisionid="57c5a03c-9095-45a4-8bb1-54f90cb4957e" lastsyncedrevisionid="57c5a03c-9095-45a4-8bb1-54f90cb4957e" lastboardhashguid="d0f34496-a6a5-16fc-241c-b0319cdc1a4e" lastpushedtime="2021-04-24T16:07:41Z" linktopcb3d="true"/>
 <plain>
 <wire x1="2.54" y1="-16.51" x2="133.33" y2="-16.51" width="0" layer="20"/>
-<wire x1="133.33" y1="-16.51" x2="133.33" y2="126.67" width="0" layer="20"/>
-<wire x1="133.33" y1="126.67" x2="2.54" y2="126.67" width="0" layer="20"/>
-<wire x1="2.54" y1="126.67" x2="2.54" y2="-16.51" width="0" layer="20"/>
+<wire x1="133.33" y1="-16.51" x2="133.33" y2="106.35" width="0" layer="20"/>
+<wire x1="133.33" y1="106.35" x2="2.54" y2="106.35" width="0" layer="20"/>
+<wire x1="2.54" y1="106.35" x2="2.54" y2="-16.51" width="0" layer="20"/>
 </plain>
 <attributes>
